File: docs/schematics/rc_power_board.kicad_sch (KiCad schematic)
At the start: 46 parts, among them J1 Battery T-plug pigtail 12AWG, J10 Radar, J11 Spare 5V, J12 IMU, J13 Shaft encoder, J14 Spare 3.3V, J2 ESC T-plug pigtail 12AWG, J3 ESC Rx lead (BEC in), J4 Servo DS3225MG, J5 Signals to ESP32, J6 USB-C > Pi 5, J7 USB-C > ESP32, J8 LIDAR-Lite v4, J9 Camera USB hub, Q1 2N7002, U1 Pololu D36V50F5 buck (req 5.1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, U2 5V buck >=4A module, TBD, U3 AP2112K-3.3 (>=300 mA LDO, TB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

Commit message: update schematic readability
Parts:
- J5: value Signals to ESP32 -> to ESP32
Other:
- moved on the sheet: J3, J4, J5
