File: docs/schematics/rc_power_board.kicad_sch (KiCad schematic)
At the start: 46 parts, among them J1 Battery T-plug pigtail 12AWG, J10 Radar, J11 Spare 5V, J12 IMU, J13 Shaft encoder, J14 Spare 3.3V, J2 ESC T-plug pigtail 12AWG, J3 ESC Rx lead (BEC in), J4 Servo DS3225MG, J5 to ESP32, J6 USB-C > Pi 5, J7 USB-C > ESP32, J8 LIDAR-Lite v4, J9 Camera USB hub, Q1 2N7002, U1 Pololu D36V50F5 buck (req 5.1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, U2 5V buck >=4A module, TBD, U3 AP2112K-3.3 (>=300 mA LDO, TB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

Commit message: Clean up power board schematic for design meeting
- Rewire each region's local nets as continuous buses (VBAT_RAW, VIN_CPU,
  VIN_SENS, LDO_IN, rail outputs) with no crossings; GND kept as symbols.
- ESC battery power moved off-board (own 12 AWG leads); remove J2/F2/
  VBAT_ESC, F1 resized to board loads (~10 A TBD), add ESC draw note.
- Archive U1 EN control: EN unconnected; remove Q1, R4, ESP_SHDN. J5 is
  now 4-pin (U1_PG, THROTTLE_PWM, STEER_PWM, GND).
- Remove radar header J10.
- Add design_overview.md meeting summary; re-export power_board_plan.md;
  update README and schematics rules.

Co-Authored-By: Claude Opus 5.5 <noreply@anthropic.com>
Claude-Session: https://claude.ai/code/session_019hn8SCZUUAVD8H8MEh7Mv7
Parts:
- removed C5: TBD >=10V, Capacitor_SMD:C_0805_2012Metric, symbol Device:C
- removed C6: TBD (filter), Capacitor_SMD:C_0805_2012Metric, symbol Device:C
- removed F2: TBD ESC branch, Fuse:Fuseholder_Blade_ATO_Littelfuse_Pudenz_2_Pin, symbol Device:Fuse
- removed H4: MountingHole_M3, MountingHole:MountingHole_3.2mm_M3, symbol Mechanical:MountingHole
- removed J10: Radar, Connector_JST:JST_XH_B2B-XH-A_1x02_P2.50mm_Vertical, symbol Connector_Generic:Conn_01x02
- removed J2: ESC T-plug pigtail 12AWG, Connector_Wire:SolderWire-2.5sqmm_1x02_P8.8mm_D2.4mm_OD4.4mm, symbol Connector_Generic:Conn_01x02
- removed J5: to ESP32, Connector_PinHeader_2.54mm:PinHeader_1x05_P2.54mm_Vertical, symbol Connector_Generic:Conn_01x05
- removed J6: USB-C > Pi 5, TerminalBlock_Phoenix:TerminalBlock_Phoenix_MKDS-1,5-2-5.08_1x02_P5.08mm_Horizontal, symbol Connector_Generic:Conn_01x02
- removed Q1: 2N7002, Package_TO_SOT_SMD:SOT-23, symbol Transistor_FET:2N7002
- removed R4: 100k, Resistor_SMD:R_0805_2012Metric, symbol Device:R
- added C2: TBD >=16V, Capacitor_SMD:C_0805_2012Metric, symbol Device:C
- added C8: 1uF TBD, Capacitor_SMD:C_0805_2012Metric, symbol Device:C
- added F4: TBD, Fuse:Fuseholder_Blade_Mini_Keystone_3568, symbol Device:Fuse
- added J3: ESC Rx lead (BEC out, throttle in), Connector_PinHeader_2.54mm:PinHeader_1x03_P2.54mm_Vertical, symbol Connector_Generic:Conn_01x03
- added J9: Camera USB hub, Connector_JST:JST_XH_B2B-XH-A_1x02_P2.50mm_Vertical, symbol Connector_Generic:Conn_01x02
- C5: renamed from F4; value TBD -> TBD >=10V; footprint Fuse:Fuseholder_Blade_Mini_Keystone_3568 -> Capacitor_SMD:C_0805_2012Metric; symbol Device:Fuse -> Device:C
- C6: renamed from J9; value Camera USB hub -> TBD filter; footprint Connector_JST:JST_XH_B2B-XH-A_1x02_P2.50mm_Vertical -> Capacitor_SMD:C_0805_2012Metric; symbol Connector_Generic:Conn_01x02 -> Device:C
- C7: value 1uF 10V TBD -> 1uF TBD
- D1: value TVS unidir. >=9V TBD -> TVS >=9V TBD
- F1: value TBD main ~30A -> TBD main ~10A
- FB1: value TBD (optional filter) -> TBD filter
- H4: renamed from C8; value 1uF 10V TBD -> MountingHole_M3; footprint Capacitor_SMD:C_0805_2012Metric -> MountingHole:MountingHole_3.2mm_M3; symbol Device:C -> Mechanical:MountingHole
- J5: renamed from J3; value ESC Rx lead (BEC in) -> Signals to ESP32; footprint Connector_PinHeader_2.54mm:PinHeader_1x03_P2.54mm_Vertical -> Connector_PinHeader_2.54mm:PinHeader_1x04_P2.54mm_Vertical; symbol Connector_Generic:Conn_01x03 -> Connector_Generic:Conn_01x04
- J6: renamed from C2; value TBD >=16V -> USB-C Pi 5; footprint Capacitor_SMD:C_0805_2012Metric -> TerminalBlock_Phoenix:TerminalBlock_Phoenix_MKDS-1,5-2-5.08_1x02_P5.08mm_Horizontal; symbol Device:C -> Connector_Generic:Conn_01x02
- J7: value USB-C > ESP32 -> USB-C ESP32
Connections:
- net +3V3_SENS: now also C8.1; no longer H4.1
- net +5V_CPU: now also J6.1 (Pin_1)
- net +5V_SENS: now also C5.1, J9.1 (Pin_1); no longer C6.1 (Pin_1)
- net +6V_BEC: now also J3.2 (Pin_2); no longer J5.2 (Pin_2)
- net GND: now also C5.2, J5.4 (Pin_4), C2.2, C8.2, J3.1 (Pin_1), J9.2 (Pin_2); no longer H4.2, J5.1 (Pin_1)
- net LDO_IN: now also C6.1
- net STEER_PWM: now also J5.3 (Pin_3)
- net THROTTLE_PWM: now also J5.2 (Pin_2), J3.3 (Pin_3); no longer J5.3 (Pin_3)
- net U1_PG: now also J5.1 (Pin_1)
- net VBAT: now also F4.1; no longer C5.1
- net VIN_CPU: now also C2.1; no longer J6.1
- net VIN_SENS: now also F4.2; no longer C5.2
- net U1_EN: no longer names the net of U1.2 (EN)
- no-connect marks 3 -> 4
Other:
- note added: "1. Battery: 2S LiPo, 6.0-8.4 V (ESC LVC cuts at 6.0 V). T-plug pigtail (12 AWG bare ends) soldered to J1 pads; pad size TBD (footprint is the 2.5 mm2 placeholder). 2. ESC is powered OFF-BOARD: battery -> ESC on its own 12 AWG leads (up to 20 A). This board carries only its own loads (about 7.3 A worst case), so F1 is sized for that, not for the motor. 3. All fuses and protection values TBD. 4. Si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"
- note added: "B ESC signals and servo"
- note added: "ESC power does NOT pass through this board: battery -> ESC on its own 12 AWG leads. J1/F1 carry only the board loads (about 7.3 A worst case at 6.4 V)."
- note added: "ESC: up to 20 A motor current (THW-1060: 60 A cont.) from the battery on its own 12 AWG leads, OFF-BOARD. Only its 3-wire receiver lead lands here (J3). J5 to ESP32: 1 U1_PG (GPIO TBD), 2 THROTTLE_PWM (GPIO5), 3 STEER_PWM (GPIO4), 4 GND. 3.3 V logic."
- note removed: "+6V_BEC comes only from the ESC BEC; never join a 5 V rail. J5: THROTTLE_PWM = GPIO5, STEER_PWM = GPIO4, U1_PG and ESP_SHDN = GPIO TBD (3.3 V logic, see region F)."
- note removed: "1. Battery: 2S LiPo, 6.0-8.4 V (ESC LVC cuts at 6.0 V). Battery and ESC use T-plug pigtails (12 AWG bare ends) soldered to J1/J2 pads; pad size TBD (12 AWG is 3.3 mm2, footprint is the 2.5 mm2 placeholder). 2. All fuses and protection values TBD; positions are proposals. 3. Single common GND; star point at J1 in layout. 4. +6V_BEC is ESC-supplied, isolated from 5 V rails. 5. Signals are 3.3 V log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"
- note removed: "B ESC and servo (servo power = ESC BEC, 6 V / 3 A)"
- note removed: "F U1 EN / PG to ESP32 (proposal, open Q13)"
- note removed: "U1 EN (D36V50F5): off below 1.2 V, on above 1.35 V. EN has a 100k pull-up to VIN inside the module (up to 8.4 V), so EN must NEVER go straight to an ESP32 GPIO (8.4 V on a 3.3 V pin while the ESP32 is off or booting). U1 also powers the ESP32, so U1 must start on its own: it stays ON by default. Proposed: ESP_SHDN high -> Q1 pulls EN low -> U1 off. This is a POWER CYCLE, not a shutdown: the ESP32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"
- note removed: "U1: all 12 module pins drawn (2x VIN, 2x VOUT, 4x GND, 2x VRP, EN, PG). VRP not used: sensor buck is fed from VBAT via F4 (decided). J6/J7: 2-wire USB-C pigtails into the Pi 5 and ESP32 USB-C inputs, so each board's own USB-C input protection is used. EN/PG control: region F."
- note removed: "U2 EN: per module datasheet, TBD. U2 footprint TBD (module pinout)."
- moved on the sheet: C5, J1
