File: docs/schematics/rc_power_board.kicad_sch (KiCad schematic)
At the start: 41 parts, among them J1 Battery T-plug pigtail 12AWG, J11 Spare 5V, J12 IMU, J13 Shaft encoder, J14 Spare 3.3V, J3 ESC Rx lead (BEC out, throttl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, J4 Servo DS3225MG, J5 Signals to ESP32, J6 USB-C Pi 5, J7 USB-C ESP32, J8 LIDAR-Lite v4, J9 Camera USB hub, U1 Pololu D36V50F5 buck (req 5.1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, U2 5V buck >=4A module, TBD, U3 AP2112K-3.3 (>=300 mA LDO, TB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

Commit message: sync schematic. all ERC checks pass
Other:
- note added: "ESP32 3V3 pin does not power these sensors (ESP32 powers nothing)."
- note removed: "ESP32 3V3 pin must not power these sensors (ESP32 powers nothing)."
