File: docs/schematics/rc_power_board.kicad_sch (KiCad schematic)
At the start: 41 parts, among them J1 Battery T-plug pigtail 12AWG, J11 Spare 5V, J12 IMU, J13 Shaft encoder, J14 Spare 3.3V, J3 ESC Rx lead (BEC out, throttl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, J4 Servo DS3225MG, J5 Signals to ESP32, J6 USB-C Pi 5, J7 USB-C ESP32, J8 LIDAR-Lite v4, J9 Camera USB hub, U1 Pololu D36V50F5 buck (req 5.1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, U2 5V buck >=4A module, TBD, U3 AP2112K-3.3 (>=300 mA LDO, TB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

Commit message: Single main fuse, BOM and fab handoff for final review
- Remove branch fuses F3/F4: one replaceable main fuse F1 (Mini/ATM blade,
  Keystone 3568 holder, type pending confirmation) protects all board
  loads; VIN_CPU/VIN_SENS merge into VBAT; drop their net-class patterns.
- Fuse verdict: standard MINI 297 (ISO 8820-3) is enough, no slow-blow
  (capacitor inrush only, motor off-board); 15 A recommended, copper
  sized for F1's rating.
- Add bom.md (proposed MPNs, verified links only, est. cost) and
  fab_handoff.md (layout/fab checklist).
- Update design_overview, README, plan (re-exported) and rules; tidy
  U2/U3 value text and mounting-hole row on the sheet.

Co-Authored-By: Claude Opus 5.5 <noreply@anthropic.com>
Claude-Session: https://claude.ai/code/session_019hn8SCZUUAVD8H8MEh7Mv7
Parts:
- removed C4: TBD >=16V, Capacitor_SMD:C_0805_2012Metric, symbol Device:C
- removed C6: TBD filter, Capacitor_SMD:C_0805_2012Metric, symbol Device:C
- removed F3: TBD, Fuse:Fuseholder_Blade_Mini_Keystone_3568, symbol Device:Fuse
- removed H2: MountingHole_M3, MountingHole:MountingHole_3.2mm_M3, symbol Mechanical:MountingHole
- added FB1: TBD filter, Inductor_SMD:L_0805_2012Metric, symbol Device:FerriteBead
- added J14: Spare 3.3V, Connector_JST:JST_XH_B2B-XH-A_1x02_P2.50mm_Vertical, symbol Connector_Generic:Conn_01x02
- C4: renamed from F4; value TBD -> TBD >=16V; footprint Fuse:Fuseholder_Blade_Mini_Keystone_3568 -> Capacitor_SMD:C_0805_2012Metric; symbol Device:Fuse -> Device:C
- C6: renamed from FB1; footprint Inductor_SMD:L_0805_2012Metric -> Capacitor_SMD:C_0805_2012Metric; symbol Device:FerriteBead -> Device:C
- F1: value TBD main ~10A -> TBD ATM mini blade 10-15A; footprint Fuse:Fuseholder_Blade_ATO_Littelfuse_Pudenz_2_Pin -> Fuse:Fuseholder_Blade_Mini_Keystone_3568
- H2: renamed from J14; value Spare 3.3V -> MountingHole_M3; footprint Connector_JST:JST_XH_B2B-XH-A_1x02_P2.50mm_Vertical -> MountingHole:MountingHole_3.2mm_M3; symbol Connector_Generic:Conn_01x02 -> Mechanical:MountingHole
Connections:
- net VIN_CPU is gone; now on net VBAT: C2.1, U1.5 (VIN), U1.6 (VIN)
- net +3V3_SENS: now also J14.1 (Pin_1); no longer H2.1 (Pin_1)
- net +5V_SENS: now also FB1.1; no longer C6.1
- net GND: now also C4.2, C6.2, J14.2 (Pin_2); no longer H2.2 (Pin_2)
- net LDO_IN: now also C6.1, FB1.2; no longer C6.2
- net VBAT: now also U2.1 (VIN)
- removed net VIN_SENS: C4.2, U2.1 (VIN)
Other:
- note added: "1. Battery: 2S LiPo, 6.0-8.4 V (ESC LVC cuts at 6.0 V). T-plug pigtail (12 AWG bare ends) soldered to J1 pads; pad size TBD (footprint is the 2.5 mm2 placeholder). 2. ESC is powered OFF-BOARD: battery -> ESC on its own 12 AWG leads (up to 20 A). This board carries only its own loads (about 7.3 A worst case; 7.8 A at 6.0 V), so F1 is sized for that, not for the motor. 3. F1 is the single replaceab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"
- note added: "ESP32 3V3 pin must not power these sensors (ESP32 powers nothing)."
- note removed: "1. Battery: 2S LiPo, 6.0-8.4 V (ESC LVC cuts at 6.0 V). T-plug pigtail (12 AWG bare ends) soldered to J1 pads; pad size TBD (footprint is the 2.5 mm2 placeholder). 2. ESC is powered OFF-BOARD: battery -> ESC on its own 12 AWG leads (up to 20 A). This board carries only its own loads (about 7.3 A worst case), so F1 is sized for that, not for the motor. 3. All fuses and protection values TBD. 4. Si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"
- note removed: "ESP32 3V3 pin does not power these sensors (ESP32 powers nothing)."
- moved on the sheet: C4
